Commit message: Align simulation stack with A2M12 and D435i sensors

File: turtlebot3_pro_description/urdf/turtlebot3_burger_pro.urdf (robot description, URDF)
Before this commit: robot turtlebot3_burger, 8 links, 7 joints
Links:
- link base_scan: mass 0.114 -> 0.19; geometry collision cylinder length=0.041 radius=0.038; visual cylinder length=0.041 radius=0.038
Joints:
- joint camera_joint: origin xyz=0.012 0 0.155 rpy=0 0 0 -> xyz=0.012 0 0.165 rpy=0 0 0

File: turtlebot3_pro_description/urdf/turtlebot3_burger_pro.urdf.xacro (robot description, xacro)
@@ -5,5 +5,5 @@
   1) 本文件是“源文件”，建议优先修改这里。
   2) turtlebot3_burger_pro.urdf 可由 xacro 展开生成，适合运行时直接加载。
-  3) 本体几何基本沿用 TB3 Burger，新增/调整了 camera_link 位姿用于你当前改装结构。
+  3) 本体几何基本沿用 TB3 Burger，传感器按 RPLIDAR A2M12 + RealSense D435i 改装结构近似。
 -->
 <robot name="turtlebot3_burger"
@@ -149,16 +149,16 @@
       <origin xyz="0 0 0.0" rpy="0 0 0"/>
       <geometry>
-        <mesh filename="package://turtlebot3_description/meshes/sensors/lds.stl" scale="0.001 0.001 0.001"/>
+        <cylinder length="0.041" radius="0.038"/>
       </geometry>
       <material name="dark"/>
     </visual>
     <collision>
-      <origin xyz="0.015 0 -0.0065" rpy="0 0 0"/>
+      <origin xyz="0 0 0" rpy="0 0 0"/>
       <geometry>
-        <cylinder length="0.0315" radius="0.055"/>
+        <cylinder length="0.041" radius="0.038"/>
       </geometry>
     </collision>
     <inertial>
-      <mass value="0.114" />
+      <mass value="0.19" />
       <origin xyz="0 0 0" />
       <inertia ixx="0.001" ixy="0.0" ixz="0.0" iyy="0.001" iyz="0.0" izz="0.001" />
@@ -169,5 +169,5 @@
     <parent link="${namespace}base_link"/>
     <child link="${namespace}camera_link"/>
-    <origin xyz="0.012 0 0.155" rpy="0 0 0"/>
+    <origin xyz="0.012 0 0.165" rpy="0 0 0"/>
   </joint>
   <link name="${namespace}camera_link">

Commit message: Adjust D435i mounting pose in simulation

File: turtlebot3_pro_description/urdf/turtlebot3_burger_pro.urdf (robot description, URDF)
Before this commit: robot turtlebot3_burger, 8 links, 7 joints
Links:
- link camera_link: geometry collision box size=0.025 0.09 0.025; visual box size=0.025 0.09 0.025
Joints:
- joint camera_joint: origin xyz=0.012 0 0.165 rpy=0 0 0 -> xyz=0.085 0 0.185 rpy=0 0 0

File: turtlebot3_pro_description/urdf/turtlebot3_burger_pro.urdf.xacro (robot description, xacro)
@@ -165,9 +165,9 @@
     </inertial>
   </link>
-  <!-- D435i 近似安装位姿：前上方 -->
+  <!-- D435i 近似安装位姿：顶层前沿，位于 RPLIDAR 前方 -->
   <joint name="${namespace}camera_joint" type="fixed">
     <parent link="${namespace}base_link"/>
     <child link="${namespace}camera_link"/>
-    <origin xyz="0.012 0 0.165" rpy="0 0 0"/>
+    <origin xyz="0.085 0 0.185" rpy="0 0 0"/>
   </joint>
   <link name="${namespace}camera_link">
@@ -175,5 +175,5 @@
       <origin xyz="0 0 0" rpy="0 0 0"/>
       <geometry>
-        <box size="0.09 0.025 0.025"/>
+        <box size="0.025 0.09 0.025"/>
       </geometry>
       <material name="blue"/>
@@ -182,5 +182,5 @@
       <origin xyz="0 0 0" rpy="0 0 0"/>
       <geometry>
-        <box size="0.09 0.025 0.025"/>
+        <box size="0.025 0.09 0.025"/>
       </geometry>
     </collision>

Commit message: Refine D435i camera mounting offset

File: turtlebot3_pro_description/urdf/turtlebot3_burger_pro.urdf (robot description, URDF)
Before this commit: robot turtlebot3_burger, 8 links, 7 joints
Joints:
- joint camera_joint: origin xyz=0.085 0 0.185 rpy=0 0 0 -> xyz=0.035 0 0.185 rpy=0 0 0

File: turtlebot3_pro_description/urdf/turtlebot3_burger_pro.urdf.xacro (robot description, xacro)
@@ -169,5 +169,5 @@
     <parent link="${namespace}base_link"/>
     <child link="${namespace}camera_link"/>
-    <origin xyz="0.085 0 0.185" rpy="0 0 0"/>
+    <origin xyz="0.035 0 0.185" rpy="0 0 0"/>
   </joint>
   <link name="${namespace}camera_link">
